File: hw/i.mx6ull-a.kicad_sch (KiCad schematic)
At the start: 1 part

Commit message: prgs
Parts:
- gave numbers to parts that had none: 1
Connections:
- net GND: now reaches U1.A1 (VSS)
- net GND: now also U1.C3 (VSS), U1.C7 (VSS), U1.E8 (VSS), U1.F6 (VSS), U1.F7 (VSS), U1.F8 (VSS), U1.F9 (VSS), U1.G3 (VSS), U1.G5 (VSS), U1.G7 (VSS), U1.H7 (VSS), U1.J5 (VSS)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
